File: Probador_Bobinas_PCB/Probador_Bobinas_PCB.kicad_pcb (KiCad board)
At the start: 2 copper layers, 61 x 74 mm, 16 parts, among them J1 WAGO_236-402, J2 WAGO_236-402, J3 PPTC041LFBN-RC, Q1 FGH60N60SFD, U1 PC817, U2 ESP32-C3_SUPERMINI_TH

Commit message: Logo SISU + designed by Ramiro en serigrafia inferior
Logo vectorizado del PNG (canal alfa) a 4 poligonos en B.SilkS, 26mm,
espejado para leerse desde abajo. Gerbers regenerados y nuevo PDF
serigrafia_ABAJO para el metodo casero.
Other:
- board text added: "designed by Ramiro"
Changed lines of the file:
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@@
 	)
 	(embedded_fonts no)
+	(gr_poly
+		(pts
+			(xy 127.630 55.472) (xy 121.769 55.472) (xy 122.056 56.650) (xy 126.251 56.650) (xy 126.452 56.736) (xy 126.394 56.880) (xy 126.193 56.937) (xy 123.177 57.454) (xy 122.516 57.713) (xy 122.344 57.914) (xy 122.286 58.287) (xy 122.602 59.609) (xy 122.775 59.954) (xy 123.292 60.327) (xy 124.010 60.499) (xy 129.986 60.499) (xy 129.670 59.178) (xy 124.987 59.178) (xy 124.814 59.092) (xy 124.901 58.948) (xy 128.434 58.345) (xy 128.836 58.201) (xy 129.124 57.943) (xy 129.210 57.483) (xy 128.836 56.104) (xy 128.463 55.730) (xy 128.090 55.558) (xy 127.630 55.472)
+		)
+		(stroke
+			(width 0.05)
+			(type solid)
+		)
+		(fill yes)
+		(layer "B.SilkS")
+	)
+	(gr_poly
+		(pts
+			(xy 121.252 55.472) (xy 118.781 55.472) (xy 120.017 60.499) (xy 122.459 60.499) (xy 121.252 55.472)
+		)
+		(stroke
+			(width 0.05)
+			(type solid)
+		)
+		(fill yes)
+		(layer "B.SilkS")
+	)
+	(gr_poly
+		(pts
+			(xy 117.373 55.472) (xy 111.541 55.472) (xy 111.829 56.650) (xy 115.994 56.650) (xy 116.167 56.736) (xy 116.109 56.880) (xy 115.937 56.937) (xy 112.892 57.454) (xy 112.317 57.684) (xy 112.059 58.029) (xy 112.030 58.287) (xy 112.490 59.896) (xy 112.748 60.155) (xy 113.064 60.327) (xy 113.811 60.499) (xy 119.643 60.499) (xy 119.327 59.178) (xy 114.759 59.178) (xy 114.587 59.034) (xy 114.989 58.891) (xy 118.207 58.345) (xy 118.810 58.000) (xy 118.925 57.770) (xy 118.925 57.425) (xy 118.551 56.075) (xy 118.149 55.702) (xy 117.373 55.472)
+		)
+		(stroke
+			(width 0.05)
+			(type solid)
+		)
+		(fill yes)
+		(layer "B.SilkS")
+	)
+	(gr_poly
+		(pts
+			(xy 111.053 55.472) (xy 108.554 55.472) (xy 109.329 58.747) (xy 109.329 58.862) (xy 109.186 58.977) (xy 107.548 58.977) (xy 107.261 58.833) (xy 106.456 55.472) (xy 104.014 55.472) (xy 104.819 59.120) (xy 104.991 59.781) (xy 105.135 60.011) (xy 105.652 60.385) (xy 106.169 60.499) (xy 111.082 60.499) (xy 111.743 60.241) (xy 111.972 59.954) (xy 112.001 59.465) (xy 111.053 55.472)
+		)
+		(stroke
+			(width 0.05)
+			(type solid)
+		)
+		(fill yes)
+		(layer "B.SilkS")
+	)
+	(gr_text "designed by Ramiro"
+		(at 117 63.2 0)
+		(layer "B.SilkS")
+		(effects
+			(font
+				(size 1.4 1.4)
+				(thickness 0.22)
+				(italic yes)
+			)
+			(justify mirror)
+		)
+	)
 )
